File: haptic-belt/haptic-belt.kicad_pcb (KiCad board)
At the start: 2 copper layers, 50.8 x 35.6 mm, 3 parts, among them J1 Conn_01x02_Male, J2 Conn_01x01, J3 Conn_01x01

Commit message: Adds manufacturing data
Other:
- board text added: "OctoPulse Belt v1 12-10-2019"
Changed lines of the file:
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@@
   (general
     (thickness 1.6)
-    (drawings 18)
+    (drawings 21)
     (tracks 10)
     (zones 0)
@@
       (net 2 "Net-(J1-Pad2)"))
   )
+  (dimension 35.56 (width 0.12) (layer B.SilkS)
+    (gr_text "35.560 mm" (at 161.925 76.2 270) (layer B.SilkS)
+      (effects (font (size 1 1) (thickness 0.15)))
+    )
+    (feature1 (pts (xy 146.05 93.98) (xy 161.241421 93.98)))
+    (feature2 (pts (xy 146.05 58.42) (xy 161.241421 58.42)))
+    (crossbar (pts (xy 160.655 58.42) (xy 160.655 93.98)))
+    (arrow1a (pts (xy 160.655 93.98) (xy 160.068579 92.853496)))
+    (arrow1b (pts (xy 160.655 93.98) (xy 161.241421 92.853496)))
+    (arrow2a (pts (xy 160.655 58.42) (xy 160.068579 59.546504)))
+    (arrow2b (pts (xy 160.655 58.42) (xy 161.241421 59.546504)))
+  )
+  (dimension 50.8 (width 0.12) (layer B.SilkS)
+    (gr_text "50.800 mm" (at 127 53.0225) (layer B.SilkS)
+      (effects (font (size 1 1) (thickness 0.15)))
+    )
+    (feature1 (pts (xy 152.4 76.2) (xy 152.4 53.706079)))
+    (feature2 (pts (xy 101.6 76.2) (xy 101.6 53.706079)))
+    (crossbar (pts (xy 101.6 54.2925) (xy 152.4 54.2925)))
+    (arrow1a (pts (xy 152.4 54.2925) (xy 151.273496 54.878921)))
+    (arrow1b (pts (xy 152.4 54.2925) (xy 151.273496 53.706079)))
+    (arrow2a (pts (xy 101.6 54.2925) (xy 102.726504 54.878921)))
+    (arrow2b (pts (xy 101.6 54.2925) (xy 102.726504 53.706079)))
+  )
+  (gr_text "OctoPulse Belt v1\n12-10-2019" (at 127 82.55) (layer B.SilkS)
+    (effects (font (size 1 1) (thickness 0.15)) (justify mirror))
+  )
   (gr_text "LRA\nor\nERM" (at 127 68.58) (layer F.SilkS)
