File: octopulse-v3/octopulse-v3.kicad_pcb (KiCad board)
At the start: 2 copper layers, 65 x 30 mm, 50 parts, among them J1 Conn_01x04_Male, J2 Conn_01x16_Male, J3 USB_C_Receptacle_USB2.0, SW1 SW_Push, SW2 SW_SPDT, U1 DRV2603, U10 ESP32-S2, U11 MPU-6050, U12 W25Q128JVS, U13 ESP-PSRAM32, U14 TP4054_[C32574], U2 DRV2603, U3 DRV2603, U4 DRV2603, U5 DRV2603, U6 DRV2603, U7 DRV2603, U8 DRV2603, U9 XC6227B331MR

Commit message: I think this is everything. Hardware complete?
Parts:
- removed the ? at (74.0, 28.0)
- removed AE1: Antenna_Loop, RF_Antenna:Texas_SWRA117D_2.4GHz_Right
- removed U12: W25Q128JVS, Package_SO:SOIC-8_5.23x5.23mm_P1.27mm
- removed U13: ESP-PSRAM32, Package_SO:SOIC-8_3.9x4.9mm_P1.27mm
- added C23: 100n, Capacitor_SMD:C_0603_1608Metric, F.Cu at (46.7, 36.1)
- added C24: 1u, Capacitor_SMD:C_0603_1608Metric, F.Cu at (46.5, 27.7)
- added C25: 100n, Capacitor_SMD:C_0603_1608Metric, F.Cu at (24.1, 37.3)
- added D1: LED, LED_SMD:LED_0603_1608Metric, F.Cu at (20.6, 26.7)
- added D2: B5819W, Diode_SMD:D_SOD-123, F.Cu at (52.3, 31.5)
- added D3: TC2020RGB-3CJH, TC2020RGB-3CJH:TC2020RGB-3CJH, F.Cu at (47.2, 31.5)
- added J4: Conn_01x02, Connector_JST:JST_PH_S2B-PH-SM4-TB_1x02-1MP_P2.00mm_Horizontal, F.Cu at (17.5, 36.1)
- added J5: Conn_01x04, Connector_JST:JST_SH_SM04B-SRSS-TB_1x04-1MP_P1.00mm_Horizontal, B.Cu at (15.7, 34.8)
- added J6: Conn_01x07, Connector_JST:JST_SH_SM07B-SRSS-TB_1x07-1MP_P1.00mm_Horizontal, F.Cu at (73.9, 35.1)
- added JP1: SolderJumper_2_Open, Jumper:SolderJumper-2_P1.3mm_Open_RoundedPad1.0x1.5mm, B.Cu at (67.3, 49.8)
- added Q1: DMG3415U, Package_TO_SOT_SMD:SOT-23, F.Cu at (53.1, 27.7)
- added Q2: DMG3415U, Package_TO_SOT_SMD:SOT-23, F.Cu at (59.2, 27.7)
- added R10: 1M, Resistor_SMD:R_0603_1608Metric, F.Cu at (24.1, 33.8)
- added R11: 1M, Resistor_SMD:R_0603_1608Metric, F.Cu at (24.1, 35.6)
- added R12: 4.7K, Resistor_SMD:R_0603_1608Metric, F.Cu at (31.2, 35.6)
- added R13: 4.7K, Resistor_SMD:R_0603_1608Metric, F.Cu at (33.0, 35.6)
- added R5: 10K, Resistor_SMD:R_0603_1608Metric, F.Cu at (24.1, 44.7)
- added R6: 1K, Resistor_SMD:R_0603_1608Metric, F.Cu at (23.6, 26.7)
- added R7: 100K, Resistor_SMD:R_0603_1608Metric, F.Cu at (50.0, 27.7)
- added R8: 100K, Resistor_SMD:R_0603_1608Metric, F.Cu at (56.1, 27.7)
- added R9: 1M, Resistor_SMD:R_0603_1608Metric, F.Cu at (48.3, 27.7)
- added SW3: SW_Push, Button_Switch_SMD:SW_SPST_PTS645, F.Cu at (18.0, 44.7)
- C20: value 100n -> 2.2n
- R2, R3: value 10K -> 5.1K
- U10: value ESP32-S2 -> ESP32-S2-WROVER; footprint Package_DFN_QFN:QFN-56-1EP_7x7mm_P0.4mm_EP5.6x5.6mm -> RF_Module:ESP32-S2-WROVER; moved to B.Cu
- U9: value XC6227B331MR -> AP2112K-3.3
- moved C21 117.6 mm to (20.6, 29.5), turned to 90 degrees
- moved U14 113.2 mm to (23.6, 29.5)
- moved R4 111.1 mm to (26.7, 26.7)
- moved C22 110.8 mm to (27.4, 28.7)
- moved SW2 81.0 mm to (65.5, 26.9), turned to 180 degrees
- moved U11 71.2 mm to (52.3, 36.1), turned to 270 degrees
- moved R2 60.2 mm to (34.8, 35.6), turned to 270 degrees
- moved C19 52.1 mm to (48.5, 36.1), turned to 90 degrees
- moved U10 50.2 mm to (57.8, 37.5), turned to 90 degrees
- moved R3 49.4 mm to (37.8, 35.6), turned to 270 degrees
- moved C18 35.0 mm to (62.2, 31.5)
- moved C20 34.7 mm to (56.6, 36.1), turned to 90 degrees
- moved C17 33.6 mm to (56.1, 31.5), turned to 90 degrees
- moved J3 21.4 mm to (36.6, 28.7), turned to 180 degrees
- moved U9 4.86 mm to (59.2, 31.5), turned to 180 degrees
Connections:
- C19 pad 1: /VDD_SPI -> Net-(C19-Pad1)
- C20 pad 1: /VDD_SPI -> Net-(C20-Pad1)
- C22 pad 1: Net-(C22-Pad1) -> VBUS
- J1 pad 1: (no net) -> /SDA
- J1 pad 2: (no net) -> /SCL
- J3 pad A1: Net-(J3-PadA1) -> GND
- J3 pad A12: Net-(J3-PadA1) -> GND
- J3 pad A4: Net-(J3-PadA4) -> VBUS
- J3 pad A5: (no net) -> Net-(J3-PadA5)
- J3 pad A6: (no net) -> /D+
- J3 pad A7: (no net) -> /D-
- J3 pad A8: (no net) -> Net-(J3-PadA8)
- J3 pad A9: Net-(J3-PadA4) -> VBUS
- J3 pad B1: Net-(J3-PadA1) -> GND
- J3 pad B12: Net-(J3-PadA1) -> GND
- J3 pad B4: Net-(J3-PadA4) -> VBUS
- J3 pad B5: (no net) -> Net-(J3-PadB5)
- J3 pad B6: (no net) -> /D+
- J3 pad B7: (no net) -> /D-
- J3 pad B8: (no net) -> Net-(J3-PadB8)
- J3 pad B9: Net-(J3-PadA4) -> VBUS
- J3 pad S1: Net-(J3-PadS1) -> GND
- R2 pad 1: /SPICS0 -> Net-(J3-PadB5)
- R2 pad 2: /VDD_SPI -> GND
- R3 pad 1: /VDD_SPI -> Net-(J3-PadA5)
- R3 pad 2: /SPICS1 -> GND
- SW2 pad 1: VDD -> GND
- SW2 pad 2: Net-(SW2-Pad2) -> Net-(Q2-Pad1)
- SW2 pad 3: GND -> Net-(SW2-Pad3)
- U10 pad 1: +3V3 -> GND
- U10 pad 10: (no net) -> /PWM5
- U10 pad 11: (no net) -> /EN4
- U10 pad 12: (no net) -> /PWM4
- U10 pad 13: (no net) -> /PWM0
- U10 pad 14: (no net) -> /EN0
- U10 pad 15: (no net) -> /PWM1
- U10 pad 16: (no net) -> /EN1
- U10 pad 17: (no net) -> /EN3
- U10 pad 18: (no net) -> /PWM3
- U10 pad 19: (no net) -> /EN2
- U10 pad 2: Net-(AE1-Pad1) -> +3V3
- U10 pad 20: +3V3 -> /PWM2
- U10 pad 21: (no net) -> /LRA
- U10 pad 22: (no net) -> /D-
- U10 pad 23: (no net) -> /D+
- U10 pad 24: (no net) -> /STATUSLED
- U10 pad 25: (no net) -> Net-(U10-Pad25)
- U10 pad 26: (no net) -> GND
- U10 pad 27: +3V3 -> Net-(U10-Pad27)
- U10 pad 28: /LRA -> Net-(U10-Pad28)
- U10 pad 29: /SPICS1 -> Net-(U10-Pad29)
- U10 pad 3: +3V3 -> /BOOT0
- U10 pad 30: /VDD_SPI -> Net-(U10-Pad30)
- U10 pad 31: /SPIHD -> Net-(U10-Pad31)
- U10 pad 32: /SPIWP -> /DBLTAP
- U10 pad 33: /SPICS0 -> /SDA
- U10 pad 34: /SPICLK -> /SCL
- U10 pad 35: /SPIQ -> /GPIO41
- U10 pad 36: /SPID -> /GPIO42
- U10 pad 37: /PWM0 -> /TXD
- U10 pad 38: /EN0 -> /RXD
- U10 pad 39: /PWM1 -> /GPIO45
- U10 pad 4: +3V3 -> /BATTMON
- U10 pad 40: /EN1 -> /IP_BTN
- U10 pad 41: /PWM2 -> /RESET
- U10 pad 42: /EN2 -> GND
- U10 pad 43: /PWM3 -> GND
- U10 pad 5: (no net) -> /EN7
- U10 pad 6: /PWM6 -> /PWM7
- U10 pad 8: /PWM7 -> /PWM6
- U10 pad 9: /EN7 -> /EN5
- U11 pad 1: (no net) -> Net-(U11-Pad1)
- U11 pad 10: (no net) -> Net-(C19-Pad1)
- U11 pad 11: (no net) -> Net-(U11-Pad11)
- U11 pad 12: (no net) -> Net-(U11-Pad12)
- U11 pad 13: (no net) -> +3V3
- U11 pad 18: (no net) -> GND
- U11 pad 20: (no net) -> Net-(C20-Pad1)
- U11 pad 23: (no net) -> /SCL
- U11 pad 24: (no net) -> /SDA
- U11 pad 6: (no net) -> Net-(U11-Pad6)
- U11 pad 7: (no net) -> Net-(U11-Pad7)
- U11 pad 8: (no net) -> +3V3
- U11 pad 9: (no net) -> Net-(U11-Pad9)
- U14 pad 1: (no net) -> Net-(D1-Pad1)
- U14 pad 4: Net-(C22-Pad1) -> VBUS
- U9 pad 3: Net-(SW2-Pad2) -> VDD
- U9 pad 4: (no net) -> Net-(U9-Pad4)
Routing:
- net +3V3: track 0.00 -> 102.2 mm, vias 0 -> 3
- net /RESET: track 0.00 -> 87.8 mm, vias 0 -> 1
- net /BATTMON: track 0.00 -> 71.4 mm, vias 0 -> 3
- net /SCL: track 0.00 -> 61.2 mm, vias 0 -> 3
- net /SDA: track 0.00 -> 59.2 mm, vias 0 -> 1
- net VBUS: track 0.00 -> 55.7 mm
- net /VBAT: track 0.00 -> 45.8 mm, vias 0 -> 2
- net /PWM0: track 0.00 -> 31.6 mm, vias 0 -> 1
- net VDD: track 78.7 -> 109.7 mm, vias 8 -> 9
- net /EN0: track 0.00 -> 27.2 mm, vias 0 -> 1
- net /SPIQ: track 26.7 -> 0.00 mm, vias 2 -> 0
- net /VDD_SPI: track 25.1 -> 0.00 mm
- net /PWM1: track 0.00 -> 22.1 mm, vias 0 -> 1
- net /SPICS1: track 20.3 -> 0.00 mm, vias 2 -> 0
- net /IP_BTN: track 11.1 -> 31.3 mm, vias 0 -> 1
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Other:
- board text added: "OctoPulse v3 2021-03-21"
- board text added: "On"
- board text added: "Reset Board"
- board text removed: "OctoPulse v2 05-11-2019"
